Commit message: updated urdf so wall is at base of bed

File: hrl_base_selection/urdf/occupied_autobed.URDF (robot description, URDF)
Before this commit: robot autobed, 26 links, 25 joints
Joints:
- joint autobed/origin_wall_joint: origin xyz=-0.75 0. 0. rpy=0 0 0 -> xyz=-0.02 0. 0. rpy=0 0 0

Commit message: thing

File: hrl_base_selection/urdf/occupied_autobed.URDF (robot description, URDF)
Before this commit: robot autobed, 26 links, 25 joints
Links:
- link autobed/bed_frame_link: geometry collision mesh filename=package://hrl_base_selection/urdf/meshes/bed_frame_link.STL; visual mesh filename=package://hrl_base_selection/urdf/meshes/bed_frame_real_exp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
Joints:
- joint autobed/origin_wall_joint: origin xyz=-0.02 0. 0. rpy=0 0 0 -> xyz=-0.12 0. 0. rpy=0 0 0
