Commit message: thing

File: hrl_base_selection/urdf/bed_and_body_expanded/robots/bed_and_body_expanded.URDF (robot description, URDF)
Before this commit: robot autobed, 28 links, 27 joints
Joints:
- joint autobed/arm_forearm_left_joint: child forearm_left_link -> autobed/forearm_left_link; parent arm_left_link -> autobed/arm_left_link
- joint autobed/arm_forearm_right_joint: child forearm_right_link -> autobed/forearm_right_link; parent arm_right_link -> autobed/arm_right_link
- joint autobed/body_arm_left_joint: child arm_left_link -> autobed/arm_left_link; parent upper_body_link -> autobed/upper_body_link
- joint autobed/body_arm_right_joint: child arm_right_link -> autobed/arm_right_link; parent upper_body_link -> autobed/upper_body_link
- joint autobed/body_quad_left_joint: child quad_left_link -> autobed/quad_left_link; parent lower_body_link -> autobed/lower_body_link
- joint autobed/body_quad_right_joint: child quad_right_link -> autobed/quad_right_link; parent lower_body_link -> autobed/lower_body_link
- joint autobed/calf_foot_left_joint: child foot_left_link -> autobed/foot_left_link; parent calf_left_link -> autobed/calf_left_link
- joint autobed/calf_foot_right_joint: child foot_right_link -> autobed/foot_right_link; parent calf_right_link -> autobed/calf_right_link
- joint autobed/forearm_hand_left_joint: child hand_left_link -> autobed/hand_left_link; parent forearm_left_link -> autobed/forearm_left_link
- joint autobed/forearm_hand_right_joint: child hand_right_link -> autobed/hand_right_link; parent forearm_right_link -> autobed/forearm_right_link
- joint autobed/head_bed_leftright_joint: child head_leftright_translation_link -> autobed/head_leftright_translation_link; parent head_rotated_to_bedframe_link -> autobed/head_rotated_to_bedframe_link
- joint autobed/head_bed_to_bedframe_joint: child head_rotated_to_bedframe_link -> autobed/head_rotated_to_bedframe_link; parent head_updown_translation_link -> autobed/head_updown_translation_link
- joint autobed/head_bed_to_worldframe_joint: child head_rotated_to_worldframe_link -> autobed/head_rotated_to_worldframe_link; parent head_rest_link -> autobed/head_rest_link
- joint autobed/head_bed_updown_joint: child head_updown_translation_link -> autobed/head_updown_translation_link; parent head_rotated_to_worldframe_link -> autobed/head_rotated_to_worldframe_link
- joint autobed/head_contact_to_head_center: child head_link -> autobed/head_link; parent head_leftright_translation_link -> autobed/head_leftright_translation_link
- joint autobed/head_neck_joint1: child neck_rotation -> autobed/neck_rotation; parent head_link -> autobed/head_link
- joint autobed/head_neck_joint2: child neck_link -> autobed/neck_link; parent neck_rotation -> autobed/neck_rotation
- joint autobed/head_rest_hinge: child head_rest_link -> autobed/head_rest_link; parent bed_frame_link -> autobed/bed_frame_link
- joint autobed/leg_rest_upper_joint: child leg_rest_upper_link -> autobed/leg_rest_upper_link; parent bed_frame_link -> autobed/bed_frame_link
- joint autobed/leg_rest_upper_lower_joint: child leg_rest_lower_link -> autobed/leg_rest_lower_link; parent leg_rest_upper_link -> autobed/leg_rest_upper_link
- joint autobed/mid_lower_body_joint: child lower_body_link -> autobed/lower_body_link; parent mid_body_link -> autobed/mid_body_link
- joint autobed/neck_body_joint: child upper_body_link -> autobed/upper_body_link; parent neck_link -> autobed/neck_link
- joint autobed/origin_wall_joint: child wall_link -> autobed/wall_link; parent base_link -> autobed/base_link
- joint autobed/quad_calf_left_joint: child calf_left_link -> autobed/calf_left_link; parent quad_left_link -> autobed/quad_left_link
- joint autobed/quad_calf_right_joint: child calf_right_link -> autobed/calf_right_link; parent quad_right_link -> autobed/quad_right_link
- joint autobed/tele_legs_joint: child bed_frame_link -> autobed/bed_frame_link; parent base_link -> autobed/base_link
- joint autobed/upper_mid_body_joint: child mid_body_link -> autobed/mid_body_link; parent upper_body_link -> autobed/upper_body_link

Commit message: pushing last changes from hydro (i hope)

File: hrl_base_selection/urdf/bed_and_body_expanded/robots/bed_and_body_expanded.URDF (robot description, URDF)
Before this commit: robot bed_and_body_v3, 28 links, 27 joints
Links:
- link arm_left_link: mass 2.60960654017703 -> None; geometry collision mesh filename=package://hrl_base_selection/urdf/bed_and_body_expanded/mes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; visual mesh filename=package://hrl_base_selection/urdf/bed_and_body_expanded/mes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
- link arm_right_link: mass 2.60960651501635 -> None; geometry collision mesh filename=package://hrl_base_selection/urdf/bed_and_body_expanded/mes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; visual mesh filename=package://hrl_base_selection/urdf/bed_and_body_expanded/mes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
- link base_link: mass 5.8260172808288 -> None; geometry collision mesh filename=package://hrl_base_selection/urdf/bed_and_body_expanded/mes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; visual mesh filename=package://hrl_base_selection/urdf/bed_and_body_expanded/mes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
- link bed_frame_link: mass 182.783 -> None; geometry collision mesh filename=package://hrl_base_selection/urdf/bed_and_body_expanded/mes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; visual mesh filename=package://hrl_base_selection/urdf/bed_and_body_expanded/mes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
- link calf_left_link: mass 3.39536669784164 -> None; geometry collision mesh filename=package://hrl_base_selection/urdf/bed_and_body_expanded/mes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; visual mesh filename=package://hrl_base_selection/urdf/bed_and_body_expanded/mes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
- link calf_right_link: mass 3.39536669784164 -> None; geometry collision mesh filename=package://hrl_base_selection/urdf/bed_and_body_expanded/mes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; visual mesh filename=package://hrl_base_selection/urdf/bed_and_body_expanded/mes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
- link foot_left_link: mass 0.615189243278472 -> None; geometry collision mesh filename=package://hrl_base_selection/urdf/bed_and_body_expanded/mes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; visual mesh filename=package://hrl_base_selection/urdf/bed_and_body_expanded/mes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
- link foot_right_link: mass 0.615189243278473 -> None; geometry collision mesh filename=package://hrl_base_selection/urdf/bed_and_body_expanded/mes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; visual mesh filename=package://hrl_base_selection/urdf/bed_and_body_expanded/mes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
- link forearm_left_link: mass 1.32173737819403 -> None; geometry collision mesh filename=package://hrl_base_selection/urdf/bed_and_body_expanded/mes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; visual mesh filename=package://hrl_base_selection/urdf/bed_and_body_expanded/mes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
- link forearm_right_link: mass 1.32173736893606 -> None; geometry collision mesh filename=package://hrl_base_selection/urdf/bed_and_body_expanded/mes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; visual mesh filename=package://hrl_base_selection/urdf/bed_and_body_expanded/mes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
- link hand_left_link: mass 1.1356241768054 -> None; geometry collision mesh filename=package://hrl_base_selection/urdf/bed_and_body_expanded/mes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; visual mesh filename=package://hrl_base_selection/urdf/bed_and_body_expanded/mes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
- link hand_right_link: mass 1.13562417680541 -> None; geometry collision mesh filename=package://hrl_base_selection/urdf/bed_and_body_expanded/mes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; visual mesh filename=package://hrl_base_selection/urdf/bed_and_body_expanded/mes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
- link head_link: mass 3.9328527892651 -> None; geometry collision mesh filename=package://hrl_base_selection/urdf/bed_and_body_expanded/mes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; visual mesh filename=package://hrl_base_selection/urdf/bed_and_body_expanded/mes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
- link head_rest_link: geometry collision mesh filename=package://hrl_base_selection/urdf/bed_and_body_expanded/mes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; visual mesh filename=package://hrl_base_selection/urdf/bed_and_body_expanded/mes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
- link leg_rest_lower_link: mass 132.5835 -> None; geometry collision mesh filename=package://hrl_base_selection/urdf/bed_and_body_expanded/mes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; visual mesh filename=package://hrl_base_selection/urdf/bed_and_body_expanded/mes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
- link leg_rest_upper_link: mass 71.0955 -> None; geometry collision mesh filename=package://hrl_base_selection/urdf/bed_and_body_expanded/mes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; visual mesh filename=package://hrl_base_selection/urdf/bed_and_body_expanded/mes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
- link lower_body_link: mass 3.76095443118537 -> None; geometry collision mesh filename=package://hrl_base_selection/urdf/bed_and_body_expanded/mes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; visual mesh filename=package://hrl_base_selection/urdf/bed_and_body_expanded/mes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
- link mid_body_link: mass 6.7659491084038 -> None; geometry collision mesh filename=package://hrl_base_selection/urdf/bed_and_body_expanded/mes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; visual mesh filename=package://hrl_base_selection/urdf/bed_and_body_expanded/mes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
- link neck_link: mass 1.53148702191926 -> None; geometry collision mesh filename=package://hrl_base_selection/urdf/bed_and_body_expanded/mes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; visual mesh filename=package://hrl_base_selection/urdf/bed_and_body_expanded/mes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
- link neck_rotation: mass 1.53148702191926 -> None; geometry collision mesh filename=package://hrl_base_selection/urdf/bed_and_body_expanded/mes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; visual mesh filename=package://hrl_base_selection/urdf/bed_and_body_expanded/mes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
- link quad_left_link: mass 6.89674952703915 -> None; geometry collision mesh filename=package://hrl_base_selection/urdf/bed_and_body_expanded/mes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; visual mesh filename=package://hrl_base_selection/urdf/bed_and_body_expanded/mes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
- link quad_right_link: mass 6.89674952703915 -> None; geometry collision mesh filename=package://hrl_base_selection/urdf/bed_and_body_expanded/mes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; visual mesh filename=package://hrl_base_selection/urdf/bed_and_body_expanded/mes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
- link upper_body_link: mass 10.994324812456 -> None; geometry collision mesh filename=package://hrl_base_selection/urdf/bed_and_body_expanded/mes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; visual mesh filename=package://hrl_base_selection/urdf/bed_and_body_expanded/mes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
- link wall_link: geometry collision mesh filename=package://hrl_base_selection/urdf/bed_and_body_expanded/mes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; visual mesh filename=package://hrl_base_selection/urdf/bed_and_body_expanded/mes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
Joints:
- joint head_rest_hinge: origin xyz=0.775 -.27375 0.26 rpy=1.5708 1.0561E-10 3.1416 -> xyz=0.794999999999999 0 0.21 rpy=1.5707963267949 0. 3.14159265358979
- joint leg_rest_upper_joint: origin xyz=1.055 -0.27375 0.05 rpy=1.5708 2.1987E-11 3.9465E-16 -> xyz=1.075 0 0 rpy=1.5708 2.1987E-11 3.9465E-16
- joint origin_wall_joint: origin xyz=-.12 0. 0 rpy=0. 0. 0. -> xyz=-.0925 0. 0 rpy=0. 0. 0.
- joint tele_legs_joint: origin xyz=-0.02 0. 0.32 rpy=0 0 0 -> xyz=-0.04 0 0.32 rpy=0 0 0
