Commit message: updates for round 2 tests at henrys

File: hrl_base_selection/urdf/bed_and_environment_henry/robots/bed_and_environment_henry.URDF (robot description, URDF)
Before this commit: robot bed_and_environment_henry, 29 links, 28 joints
Links:
- removed link autobed/head_leftright_translation_link
- removed link autobed/head_rotated_to_bedframe_link
- removed link autobed/head_rotated_to_worldframe_link
- removed link autobed/head_updown_in_bedframe_link
- removed link autobed/head_updown_translation_link
- removed link autobed/neck_rotation
- added link autobed/head_roty_link
- added link autobed/head_rotz_link
- added link autobed/neck_base_link
- added link autobed/neck_rotated_to_bedframe_link
- added link autobed/neck_rotated_to_worldframe_link
- added link autobed/neck_tilt_link
- added link autobed/neck_top_rotated_link
- added link autobed/neck_twist_link
- added link autobed/neck_updown_bedframe_translation_link
- added link autobed/neck_updown_worldframe_translation_link
Joints:
- removed joint autobed/head_bed_leftright_joint
- removed joint autobed/head_bed_to_bedframe_joint
- removed joint autobed/head_bed_to_worldframe_joint
- removed joint autobed/head_bed_updown_joint
- removed joint autobed/head_contact_to_head_center
- removed joint autobed/head_neck_joint1
- removed joint autobed/head_neck_joint2
- removed joint autobed/head_updown_bedframe_translation_joint
- added joint autobed/bed_neck_base_leftright_joint: type prismatic, parent autobed/neck_updown_bedframe_translation_link, child autobed/neck_base_link, origin xyz=0 0 0 rpy=0 3.14159 0, axis 0 0 -1, limit lower=-2 upper=2 effort=0 velocity=0
- added joint autobed/bed_neck_base_updown_bedframe_joint: type prismatic, parent autobed/neck_rotated_to_bedframe_link, child autobed/neck_updown_bedframe_translation_link, origin xyz=0.0 0.0 0 rpy=0. 0. 0., axis -1 0 0, limit lower=-2 upper=2 effort=0 velocity=0
- added joint autobed/bed_neck_to_bedframe_joint: type revolute, parent autobed/neck_updown_worldframe_translation_link, child autobed/neck_rotated_to_bedframe_link, origin xyz=0.0 0.0 0 rpy=0. 0. 0., axis 0 0 1, limit lower=-2 upper=2 effort=0 velocity=0
- added joint autobed/bed_neck_worldframe_updown_joint: type prismatic, parent autobed/neck_rotated_to_worldframe_link, child autobed/neck_updown_worldframe_translation_link, origin xyz=0.0 0.0 0 rpy=0.0 0.0 0.0, axis -1 0 0, limit lower=-2 upper=2 effort=0 velocity=0
- added joint autobed/headrest_bed_to_worldframe_joint: type revolute, parent autobed/head_rest_link, child autobed/neck_rotated_to_worldframe_link, origin xyz=0.25949 0.1 0 rpy=0. 0. 0., axis 0 0 1, limit lower=-2 upper=2 effort=0 velocity=0
- added joint autobed/neck_head_rotx_joint: type revolute, parent autobed/head_rotz_link, child autobed/head_link, origin xyz=0 0 0 rpy=0 0 0, axis 1 0 0, limit lower=-2 upper=2 effort=0 velocity=0
- added joint autobed/neck_head_roty_joint: type revolute, parent autobed/neck_top_rotated_link, child autobed/head_roty_link, origin xyz=0.0154 0 0.07779 rpy=0 0 0, axis 0 1 0, limit lower=-2 upper=2 effort=0 velocity=0
- added joint autobed/neck_head_rotz_joint: type revolute, parent autobed/head_roty_link, child autobed/head_rotz_link, origin xyz=0 0 0 rpy=0 0 0, axis 0 0 1, limit lower=-2 upper=2 effort=0 velocity=0
- added joint autobed/neck_rotation_fixed_joint: type fixed, parent autobed/neck_link, child autobed/neck_top_rotated_link, origin xyz=0 0 0 rpy=-1.570796 0 1.570796, axis 0 0 1, limit lower=-2 upper=2 effort=0 velocity=0
- added joint autobed/neck_tilt_joint: type revolute, parent autobed/neck_twist_link, child autobed/neck_tilt_link, origin xyz=0.0 0.0 0 rpy=0. 0. 0., axis 0 0 -1, limit lower=-2 upper=2 effort=0 velocity=0
- added joint autobed/neck_to_neck_top_joint: type fixed, parent autobed/neck_tilt_link, child autobed/neck_link, origin xyz=-0.07239 0 0 rpy=0 0 0
- added joint autobed/neck_twist_joint: type revolute, parent autobed/neck_base_link, child autobed/neck_twist_link, origin xyz=0.0 0.0 0 rpy=0. 0. 0., axis 1 0 0, limit lower=-2 upper=2 effort=0 velocity=0
- joint autobed/arm_forearm_left_joint: origin xyz=0.28174 -0.0106 -0.04953 rpy=1.1849E-16 -8.3419E-14 -1.6268E-27 -> xyz=0.28174 -0.0106 -0.04953 rpy=0 0 0
- joint autobed/arm_forearm_right_joint: origin xyz=0.28194 0 0.04953 rpy=2.6089E-19 -8.3342E-14 0.037607 -> xyz=0.28194 0 0.04953 rpy=0 0 0
- joint autobed/body_arm_left_joint: origin xyz=0.09652 0 -0.17526 rpy=2.6872E-15 8.287E-14 0.033074 -> xyz=0.09652 0 -0.17526 rpy=0 0 0
- joint autobed/body_arm_right_joint: origin xyz=0.09652 0 0.17526 rpy=-3.0757E-16 8.2843E-14 -0.0045332 -> xyz=0.09652 0 0.17526 rpy=0 0 0
- joint autobed/body_quad_left_joint: origin xyz=0.05207 0 -0.08636 rpy=-3.1554E-30 -3.1554E-30 -2.7756E-17 -> xyz=0.05207 0 -0.08636 rpy=0 0 -.25
- joint autobed/body_quad_right_joint: origin xyz=0.05207 0 0.08636 rpy=-3.1554E-30 -3.1554E-30 -2.7756E-17 -> xyz=0.05207 0 0.08636 rpy=0 0 -.25
- joint autobed/calf_foot_left_joint: origin xyz=-0.41279 -0.03188 0 rpy=2.4608E-16 9.411E-16 0.077076 -> xyz=-0.41279 -0.03188 0 rpy=0 0 0.09
- joint autobed/calf_foot_right_joint: origin xyz=-0.41279 -0.03188 0 rpy=3.3137E-27 3.7799E-26 0.077076 -> xyz=-0.41279 -0.03188 0 rpy=0 0 0.09
- joint autobed/forearm_hand_left_joint: origin xyz=0.25146 0 0 rpy=1.3447E-16 8.3999E-14 1.6283E-27 -> xyz=0.25146 0 0 rpy=0 0 0
- joint autobed/forearm_hand_right_joint: origin xyz=0.25146 0 0 rpy=1.9364E-14 8.3335E-14 1.6151E-27 -> xyz=0.25146 0 0 rpy=0 0 0
- joint autobed/mid_lower_body_joint: axis 0 0 -1 -> 0 0 1; origin xyz=0.15113 0 0 rpy=-4.3091E-16 1.669E-15 -0.57779 -> xyz=0.15113 0 0 rpy=0 0 0
- joint autobed/neck_body_joint: origin xyz=0.07239 0 0 rpy=-8.8242E-17 -8.2927E-14 0.66506 -> xyz=0.00 0 0 rpy=0 0 0; parent autobed/neck_link -> autobed/neck_base_link
- joint autobed/quad_calf_left_joint: origin xyz=0.41218 0.11044 0 rpy=3.1416 8.5469E-14 -2.8798 -> xyz=0.41218 0.11044 0 rpy=3.14159 0 3.43
- joint autobed/quad_calf_right_joint: origin xyz=0.41218 0.11044 0 rpy=3.1416 8.5225E-14 -2.8798 -> xyz=0.41218 0.11044 0 rpy=3.14159 0 3.43
- joint autobed/upper_mid_body_joint: axis 0 0 -1 -> 0 0 1; origin xyz=0.35052 0 0 rpy=2.8327E-14 7.7949E-14 0.34907 -> xyz=0.35052 0 0 rpy=0 0 0

File: hrl_base_selection/urdf/wheelchair_henry/robots/wheelchair_henry.URDF (robot description, URDF)
Before this commit: robot wheelchair_henry, 19 links, 18 joints
Links:
- removed link wheelchair/neck_rotation
- added link wheelchair/head_roty_link
- added link wheelchair/head_rotz_link
- added link wheelchair/neck_base_link
- added link wheelchair/neck_tilt_link
- added link wheelchair/neck_top_rotated_link
- added link wheelchair/neck_twist_link
- link wheelchair/arm_left_link: geometry collision mesh filename=package://hrl_base_selection/urdf/bed_and_environment_henry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; visual mesh filename=package://hrl_base_selection/urdf/bed_and_environment_henry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
- link wheelchair/arm_right_link: geometry collision mesh filename=package://hrl_base_selection/urdf/bed_and_environment_henry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; visual mesh filename=package://hrl_base_selection/urdf/bed_and_environment_henry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
- link wheelchair/calf_left_link: geometry collision mesh filename=package://hrl_base_selection/urdf/bed_and_environment_henry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; visual mesh filename=package://hrl_base_selection/urdf/bed_and_environment_henry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
- link wheelchair/calf_right_link: geometry collision mesh filename=package://hrl_base_selection/urdf/bed_and_environment_henry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; visual mesh filename=package://hrl_base_selection/urdf/bed_and_environment_henry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
- link wheelchair/foot_left_link: geometry collision mesh filename=package://hrl_base_selection/urdf/bed_and_environment_henry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; visual mesh filename=package://hrl_base_selection/urdf/bed_and_environment_henry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
- link wheelchair/foot_right_link: geometry collision mesh filename=package://hrl_base_selection/urdf/bed_and_environment_henry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; visual mesh filename=package://hrl_base_selection/urdf/bed_and_environment_henry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
- link wheelchair/forearm_left_link: geometry collision mesh filename=package://hrl_base_selection/urdf/bed_and_environment_henry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; visual mesh filename=package://hrl_base_selection/urdf/bed_and_environment_henry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
- link wheelchair/forearm_right_link: geometry collision mesh filename=package://hrl_base_selection/urdf/bed_and_environment_henry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; visual mesh filename=package://hrl_base_selection/urdf/bed_and_environment_henry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
- link wheelchair/hand_left_link: geometry collision mesh filename=package://hrl_base_selection/urdf/bed_and_environment_henry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; visual mesh filename=package://hrl_base_selection/urdf/bed_and_environment_henry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
- link wheelchair/hand_right_link: geometry collision mesh filename=package://hrl_base_selection/urdf/bed_and_environment_henry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; visual mesh filename=package://hrl_base_selection/urdf/bed_and_environment_henry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
- link wheelchair/head_link: geometry collision mesh filename=package://hrl_base_selection/urdf/bed_and_environment_henry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; visual mesh filename=package://hrl_base_selection/urdf/bed_and_environment_henry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
- link wheelchair/lower_body_link: geometry collision mesh filename=package://hrl_base_selection/urdf/bed_and_environment_henry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; visual mesh filename=package://hrl_base_selection/urdf/bed_and_environment_henry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
- link wheelchair/mid_body_link: geometry collision mesh filename=package://hrl_base_selection/urdf/bed_and_environment_henry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; visual mesh filename=package://hrl_base_selection/urdf/bed_and_environment_henry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
- link wheelchair/neck_link: geometry collision mesh filename=package://hrl_base_selection/urdf/bed_and_environment_henry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; visual mesh filename=package://hrl_base_selection/urdf/bed_and_environment_henry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
- link wheelchair/quad_left_link: geometry collision mesh filename=package://hrl_base_selection/urdf/bed_and_environment_henry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; visual mesh filename=package://hrl_base_selection/urdf/bed_and_environment_henry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
- link wheelchair/quad_right_link: geometry collision mesh filename=package://hrl_base_selection/urdf/bed_and_environment_henry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; visual mesh filename=package://hrl_base_selection/urdf/bed_and_environment_henry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
- link wheelchair/upper_body_link: geometry collision mesh filename=package://hrl_base_selection/urdf/bed_and_environment_henry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; visual mesh filename=package://hrl_base_selection/urdf/bed_and_environment_henry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
Joints:
- removed joint wheelchair/head_neck_joint1
- removed joint wheelchair/head_neck_joint2
- removed joint wheelchair/origin_to_base_joint
- added joint wheelchair/neck_head_rotx_joint: type revolute, parent wheelchair/head_rotz_link, child wheelchair/head_link, origin xyz=0 0 0 rpy=0 0 0, axis 1 0 0, limit lower=-2 upper=2 effort=0 velocity=0
- added joint wheelchair/neck_head_roty_joint: type revolute, parent wheelchair/neck_top_rotated_link, child wheelchair/head_roty_link, origin xyz=0.0154 0 0.07779 rpy=0 0 0, axis 0 1 0, limit lower=-2 upper=2 effort=0 velocity=0
- added joint wheelchair/neck_head_rotz_joint: type revolute, parent wheelchair/head_roty_link, child wheelchair/head_rotz_link, origin xyz=0 0 0 rpy=0 0 0, axis 0 0 1, limit lower=-2 upper=2 effort=0 velocity=0
- added joint wheelchair/neck_rotation_fixed_joint: type fixed, parent wheelchair/neck_link, child wheelchair/neck_top_rotated_link, origin xyz=0 0 0 rpy=-1.570796 0 1.570796, axis 0 0 1, limit lower=-2 upper=2 effort=0 velocity=0
- added joint wheelchair/neck_tilt_joint: type revolute, parent wheelchair/neck_twist_link, child wheelchair/neck_tilt_link, origin xyz=0.0 0.0 0 rpy=0. 0. 0., axis 0 0 -1, limit lower=-2 upper=2 effort=0 velocity=0
- added joint wheelchair/neck_to_neck_top_joint: type fixed, parent wheelchair/neck_tilt_link, child wheelchair/neck_link, origin xyz=-0.07239 0 0 rpy=0 0 0
- added joint wheelchair/neck_twist_joint: type revolute, parent wheelchair/neck_base_link, child wheelchair/neck_twist_link, origin xyz=0.0 0.0 0 rpy=0. 0. 0., axis 1 0 0, limit lower=-2 upper=2 effort=0 velocity=0
- added joint wheelchair/origin_to_neck_base_joint: type fixed, parent wheelchair/base_link, child wheelchair/neck_base_link, origin xyz=0.332 0 1.25 rpy=1.570795 1.570795 0
- joint wheelchair/arm_forearm_left_joint: origin xyz=0.28174 -0.0106 -0.04953 rpy=1.1849E-16 -8.3419E-14 -1.6268E-27 -> xyz=0.28174 -0.0106 -0.04953 rpy=0 0 0
- joint wheelchair/arm_forearm_right_joint: origin xyz=0.28194 0 0.04953 rpy=2.6089E-19 -8.3342E-14 0.037607 -> xyz=0.28194 0 0.04953 rpy=0 0 0
- joint wheelchair/body_arm_left_joint: origin xyz=0.09652 0 -0.17526 rpy=2.6872E-15 8.287E-14 0.033074 -> xyz=0.09652 0 -0.17526 rpy=0 0 0
- joint wheelchair/body_arm_right_joint: origin xyz=0.09652 0 0.17526 rpy=-3.0757E-16 8.2843E-14 -0.0045332 -> xyz=0.09652 0 0.17526 rpy=0 0 0
- joint wheelchair/body_quad_left_joint: origin xyz=0.05207 0 -0.08636 rpy=-3.1554E-30 -3.1554E-30 -2.7756E-17 -> xyz=0.05207 0 -0.08636 rpy=0 0 -.25
- joint wheelchair/body_quad_right_joint: origin xyz=0.05207 0 0.08636 rpy=-3.1554E-30 -3.1554E-30 -2.7756E-17 -> xyz=0.05207 0 0.08636 rpy=0 0 -.25
- joint wheelchair/calf_foot_left_joint: origin xyz=-0.41279 -0.03188 0 rpy=2.4608E-16 9.411E-16 0.077076 -> xyz=-0.41279 -0.03188 0 rpy=0 0 0.09
- joint wheelchair/calf_foot_right_joint: origin xyz=-0.41279 -0.03188 0 rpy=3.3137E-27 3.7799E-26 0.077076 -> xyz=-0.41279 -0.03188 0 rpy=0 0 0.09
- joint wheelchair/forearm_hand_left_joint: origin xyz=0.25146 0 0 rpy=1.3447E-16 8.3999E-14 1.6283E-27 -> xyz=0.25146 0 0 rpy=0 0 0
- joint wheelchair/forearm_hand_right_joint: origin xyz=0.25146 0 0 rpy=1.9364E-14 8.3335E-14 1.6151E-27 -> xyz=0.25146 0 0 rpy=0 0 0
- joint wheelchair/mid_lower_body_joint: axis 0 0 -1 -> 0 0 1; origin xyz=0.15113 0 0 rpy=-4.3091E-16 1.669E-15 -0.57779 -> xyz=0.15113 0 0 rpy=0 0 0
- joint wheelchair/neck_body_joint: origin xyz=0.07239 0 0 rpy=-8.8242E-17 -8.2927E-14 0.66506 -> xyz=0.00 0 0 rpy=0 0 0; parent wheelchair/neck_link -> wheelchair/neck_base_link
- joint wheelchair/quad_calf_left_joint: origin xyz=0.41218 0.11044 0 rpy=3.1416 8.5469E-14 -2.8798 -> xyz=0.41218 0.11044 0 rpy=3.14159 0 3.43
- joint wheelchair/quad_calf_right_joint: origin xyz=0.41218 0.11044 0 rpy=3.1416 8.5225E-14 -2.8798 -> xyz=0.41218 0.11044 0 rpy=3.14159 0 3.43
- joint wheelchair/upper_mid_body_joint: axis 0 0 -1 -> 0 0 1; origin xyz=0.35052 0 0 rpy=2.8327E-14 7.7949E-14 0.34907 -> xyz=0.35052 0 0 rpy=0 0 0
