Commit message: added right transform to distance check

File: hrl_base_selection/urdf/bed_and_environment_henry/robots/bed_and_environment_henry_head_position.URDF (robot description, URDF)
Before this commit: robot wheelchair_henry, 24 links, 23 joints
Links:
- removed link wheelchair/arm_left_link
- removed link wheelchair/arm_right_link
- removed link wheelchair/base_link
- removed link wheelchair/calf_left_link
- removed link wheelchair/calf_right_link
- removed link wheelchair/foot_left_link
- removed link wheelchair/foot_right_link
- removed link wheelchair/forearm_left_link
- removed link wheelchair/forearm_right_link
- removed link wheelchair/hand_left_link
- removed link wheelchair/hand_right_link
- removed link wheelchair/head_link
- removed link wheelchair/head_roty_link
- removed link wheelchair/head_rotz_link
- removed link wheelchair/lower_body_link
- removed link wheelchair/mid_body_link
- removed link wheelchair/neck_base_link
- removed link wheelchair/neck_link
- removed link wheelchair/neck_tilt_link
- removed link wheelchair/neck_top_rotated_link
- removed link wheelchair/neck_twist_link
- removed link wheelchair/quad_left_link
- removed link wheelchair/quad_right_link
- removed link wheelchair/upper_body_link
- added link autobed/arm_left_link; collision mesh filename=package://hrl_base_selection/urdf/bed_and_environment_henry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; visual mesh filename=package://hrl_base_selection/urdf/bed_and_environment_henry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
- added link autobed/arm_right_link; collision mesh filename=package://hrl_base_selection/urdf/bed_and_environment_henry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; visual mesh filename=package://hrl_base_selection/urdf/bed_and_environment_henry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
- added link autobed/base_link, mass 6.1860172808288; collision mesh filename=package://hrl_base_selection/urdf/bed_and_environment_henry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; visual mesh filename=package://hrl_base_selection/urdf/bed_and_environment_henry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
- added link autobed/bed_frame_link, mass 298.525793737685; collision mesh filename=package://hrl_base_selection/urdf/bed_and_environment_henry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; visual mesh filename=package://hrl_base_selection/urdf/bed_and_environment_henry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
- added link autobed/calf_left_link; collision mesh filename=package://hrl_base_selection/urdf/bed_and_environment_henry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; visual mesh filename=package://hrl_base_selection/urdf/bed_and_environment_henry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
- added link autobed/calf_right_link; collision mesh filename=package://hrl_base_selection/urdf/bed_and_environment_henry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; visual mesh filename=package://hrl_base_selection/urdf/bed_and_environment_henry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
- added link autobed/foot_left_link; collision mesh filename=package://hrl_base_selection/urdf/bed_and_environment_henry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; visual mesh filename=package://hrl_base_selection/urdf/bed_and_environment_henry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
- added link autobed/foot_right_link; collision mesh filename=package://hrl_base_selection/urdf/bed_and_environment_henry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; visual mesh filename=package://hrl_base_selection/urdf/bed_and_environment_henry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
- added link autobed/forearm_left_link; collision mesh filename=package://hrl_base_selection/urdf/bed_and_environment_henry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; visual mesh filename=package://hrl_base_selection/urdf/bed_and_environment_henry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
- added link autobed/forearm_right_link; collision mesh filename=package://hrl_base_selection/urdf/bed_and_environment_henry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; visual mesh filename=package://hrl_base_selection/urdf/bed_and_environment_henry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
- added link autobed/hand_left_link; collision mesh filename=package://hrl_base_selection/urdf/bed_and_environment_henry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; visual mesh filename=package://hrl_base_selection/urdf/bed_and_environment_henry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
- added link autobed/hand_right_link; collision mesh filename=package://hrl_base_selection/urdf/bed_and_environment_henry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; visual mesh filename=package://hrl_base_selection/urdf/bed_and_environment_henry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
- added link autobed/head_leftright_translation_link
- added link autobed/head_link; collision mesh filename=package://hrl_base_selection/urdf/bed_and_environment_henry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; visual mesh filename=package://hrl_base_selection/urdf/bed_and_environment_henry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
- added link autobed/head_rest_link, mass 158.265573279578; collision mesh filename=package://hrl_base_selection/urdf/bed_and_environment_henry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; visual mesh filename=package://hrl_base_selection/urdf/bed_and_environment_henry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
- added link autobed/head_rotated_to_bedframe_link
- added link autobed/head_rotated_to_worldframe_link
- added link autobed/head_updown_in_bedframe_link
- added link autobed/head_updown_translation_link
- added link autobed/leg_rest_lower, mass 124.8975; collision mesh filename=package://hrl_base_selection/urdf/bed_and_environment_henry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; visual mesh filename=package://hrl_base_selection/urdf/bed_and_environment_henry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
- added link autobed/leg_rest_upper, mass 71.0955000000001; collision mesh filename=package://hrl_base_selection/urdf/bed_and_environment_henry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; visual mesh filename=package://hrl_base_selection/urdf/bed_and_environment_henry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
- added link autobed/lower_body_link; collision mesh filename=package://hrl_base_selection/urdf/bed_and_environment_henry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; visual mesh filename=package://hrl_base_selection/urdf/bed_and_environment_henry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
- added link autobed/mid_body_link; collision mesh filename=package://hrl_base_selection/urdf/bed_and_environment_henry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; visual mesh filename=package://hrl_base_selection/urdf/bed_and_environment_henry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
- added link autobed/neck_link; collision mesh filename=package://hrl_base_selection/urdf/bed_and_environment_henry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; visual mesh filename=package://hrl_base_selection/urdf/bed_and_environment_henry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
- added link autobed/neck_rotation; collision mesh filename=package://hrl_base_selection/urdf/bed_and_environment_henry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; visual mesh filename=package://hrl_base_selection/urdf/bed_and_environment_henry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
- added link autobed/quad_left_link; collision mesh filename=package://hrl_base_selection/urdf/bed_and_environment_henry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; visual mesh filename=package://hrl_base_selection/urdf/bed_and_environment_henry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
- added link autobed/quad_right_link; collision mesh filename=package://hrl_base_selection/urdf/bed_and_environment_henry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; visual mesh filename=package://hrl_base_selection/urdf/bed_and_environment_henry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
- added link autobed/upper_body_link; collision mesh filename=package://hrl_base_selection/urdf/bed_and_environment_henry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; visual mesh filename=package://hrl_base_selection/urdf/bed_and_environment_henry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
- added link autobed/wall_link, mass 3480.34879229199; collision mesh filename=package://hrl_base_selection/urdf/bed_and_environment_henry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; visual mesh filename=package://hrl_base_selection/urdf/bed_and_environment_henry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
Joints:
- removed joint wheelchair/arm_forearm_left_joint
- removed joint wheelchair/arm_forearm_right_joint
- removed joint wheelchair/body_arm_left_joint
- removed joint wheelchair/body_arm_right_joint
- removed joint wheelchair/body_quad_left_joint
- removed joint wheelchair/body_quad_right_joint
- removed joint wheelchair/calf_foot_left_joint
- removed joint wheelchair/calf_foot_right_joint
- removed joint wheelchair/forearm_hand_left_joint
- removed joint wheelchair/forearm_hand_right_joint
- removed joint wheelchair/mid_lower_body_joint
- removed joint wheelchair/neck_body_joint
- removed joint wheelchair/neck_head_rotx_joint
- removed joint wheelchair/neck_head_roty_joint
- removed joint wheelchair/neck_head_rotz_joint
- removed joint wheelchair/neck_rotation_fixed_joint
- removed joint wheelchair/neck_tilt_joint
- removed joint wheelchair/neck_to_neck_top_joint
- removed joint wheelchair/neck_twist_joint
- removed joint wheelchair/origin_to_neck_base_joint
- removed joint wheelchair/quad_calf_left_joint
- removed joint wheelchair/quad_calf_right_joint
- removed joint wheelchair/upper_mid_body_joint
- added joint autobed/arm_forearm_left_joint: type revolute, parent autobed/arm_left_link, child autobed/forearm_left_link, origin xyz=0.28174 -0.0106 -0.04953 rpy=1.1849E-16 -8.3419E-14 -1.6268E-27, axis 0 0 1, limit lower=-3 upper=3 effort=0 velocity=0
- added joint autobed/arm_forearm_right_joint: type revolute, parent autobed/arm_right_link, child autobed/forearm_right_link, origin xyz=0.28194 0 0.04953 rpy=2.6089E-19 -8.3342E-14 0.037607, axis 0 0 1, limit lower=-3 upper=3 effort=0 velocity=0
- added joint autobed/body_arm_left_joint: type revolute, parent autobed/upper_body_link, child autobed/arm_left_link, origin xyz=0.09652 0 -0.17526 rpy=2.6872E-15 8.287E-14 0.033074, axis 0 0 1, limit lower=-3 upper=3 effort=0 velocity=0
- added joint autobed/body_arm_right_joint: type revolute, parent autobed/upper_body_link, child autobed/arm_right_link, origin xyz=0.09652 0 0.17526 rpy=-3.0757E-16 8.2843E-14 -0.0045332, axis 0 0 1, limit lower=-3 upper=3 effort=0 velocity=0
- added joint autobed/body_quad_left_joint: type revolute, parent autobed/lower_body_link, child autobed/quad_left_link, origin xyz=0.05207 0 -0.08636 rpy=-3.1554E-30 -3.1554E-30 -2.7756E-17, axis 0 0 1, limit lower=-3. upper=3. effort=0 velocity=0
- added joint autobed/body_quad_right_joint: type revolute, parent autobed/lower_body_link, child autobed/quad_right_link, origin xyz=0.05207 0 0.08636 rpy=-3.1554E-30 -3.1554E-30 -2.7756E-17, axis 0 0 1, limit lower=-3 upper=3 effort=0 velocity=0
- added joint autobed/calf_foot_left_joint: type revolute, parent autobed/calf_left_link, child autobed/foot_left_link, origin xyz=-0.41279 -0.03188 0 rpy=2.4608E-16 9.411E-16 0.077076, axis 0 0 1, limit lower=-3. upper=3. effort=0 velocity=0
- added joint autobed/calf_foot_right_joint: type revolute, parent autobed/calf_right_link, child autobed/foot_right_link, origin xyz=-0.41279 -0.03188 0 rpy=3.3137E-27 3.7799E-26 0.077076, axis 0 0 1, limit lower=-3 upper=3 effort=0 velocity=0
- added joint autobed/forearm_hand_left_joint: type revolute, parent autobed/forearm_left_link, child autobed/hand_left_link, origin xyz=0.25146 0 0 rpy=1.3447E-16 8.3999E-14 1.6283E-27, axis 0 0 1, limit lower=-3 upper=3 effort=0 velocity=0
- added joint autobed/forearm_hand_right_joint: type revolute, parent autobed/forearm_right_link, child autobed/hand_right_link, origin xyz=0.25146 0 0 rpy=1.9364E-14 8.3335E-14 1.6151E-27, axis 0 0 1, limit lower=-3 upper=3 effort=0 velocity=0
- added joint autobed/head_bed_leftright_joint: type prismatic, parent autobed/head_updown_in_bedframe_link, child autobed/head_leftright_translation_link, origin xyz=0 0 0 rpy=0.0 0.0 1.570796, axis 0 0 1, limit lower=-2 upper=2 effort=0 velocity=0
- added joint autobed/head_bed_to_bedframe_joint: type revolute, parent autobed/head_updown_translation_link, child autobed/head_rotated_to_bedframe_link, origin xyz=0.0 0.0 0 rpy=0. 0. 0., axis 0 0 1, limit lower=-2 upper=2 effort=0 velocity=0
- added joint autobed/head_bed_to_worldframe_joint: type revolute, parent autobed/head_rest_link, child autobed/head_rotated_to_worldframe_link, origin xyz=0.40949 0.05 0 rpy=0. 0. 0., axis 0 0 1, limit lower=-2 upper=2 effort=0 velocity=0
- added joint autobed/head_bed_updown_joint: type prismatic, parent autobed/head_rotated_to_worldframe_link, child autobed/head_updown_translation_link, origin xyz=0.0 0.0 0 rpy=0.0 0.0 0.0, axis -1 0 0, limit lower=-2 upper=2 effort=0 velocity=0
- added joint autobed/head_contact_to_head_center: type revolute, parent autobed/head_leftright_translation_link, child autobed/head_link, origin xyz=0.091171 0.037577 0 rpy=1.5708 0 0.2618, axis 0 -1 0, limit lower=-2 upper=2 effort=0 velocity=0
- added joint autobed/head_neck_joint1: type revolute, parent autobed/head_link, child autobed/neck_rotation, origin xyz=-0.0254 0 -0.08509 rpy=-1.5708 1.1345 -3.1416, axis 0 0 -1, limit lower=-2 upper=2 effort=0 velocity=0
- added joint autobed/head_neck_joint2: type revolute, parent autobed/neck_rotation, child autobed/neck_link, origin xyz=0 0 0 rpy=0 3.1554E-30 0, axis 0 0 1, limit lower=-2 upper=2 effort=0 velocity=0
- added joint autobed/head_rest_hinge: type revolute, parent autobed/bed_frame_link, child autobed/head_rest_link, origin xyz=0.795 0 0.21 rpy=1.5708 0 -3.1416, axis 0 0 1, limit lower=-2 upper=2 effort=0 velocity=0
- added joint autobed/head_updown_bedframe_translation_joint: type prismatic, parent autobed/head_rotated_to_bedframe_link, child autobed/head_updown_in_bedframe_link, origin xyz=0.0 0.0 0 rpy=0. 0. 0., axis -1 0 0, limit lower=-2 upper=2 effort=0 velocity=0
- added joint autobed/leg_rest_lower_hinge: type revolute, parent autobed/leg_rest_upper, child autobed/leg_rest_lower, origin xyz=0.37 0 0 rpy=8.4655E-16 -2.4744E-16 -1.8316E-16, axis 0 0 -1, limit lower=-2 upper=2 effort=0 velocity=0
- added joint autobed/leg_rest_upper_hinge: type revolute, parent autobed/bed_frame_link, child autobed/leg_rest_upper, origin xyz=1.075 0 0 rpy=1.5708 -1.8438E-16 7.6543E-16, axis 0 0 1, limit lower=-2 upper=2 effort=0 velocity=0
- added joint autobed/mid_lower_body_joint: type revolute, parent autobed/mid_body_link, child autobed/lower_body_link, origin xyz=0.15113 0 0 rpy=-4.3091E-16 1.669E-15 -0.57779, axis 0 0 -1, limit lower=-2 upper=2 effort=0 velocity=0
- added joint autobed/neck_body_joint: type revolute, parent autobed/neck_link, child autobed/upper_body_link, origin xyz=0.07239 0 0 rpy=-8.8242E-17 -8.2927E-14 0.66506, axis 0 0 -1, limit lower=-2 upper=2 effort=0 velocity=0
- added joint autobed/origin_wall_joint: type fixed, parent autobed/base_link, child autobed/wall_link, origin xyz=-0.12155 -0.0043316 0 rpy=0 0 -0.053897, axis 0 0 0
- added joint autobed/quad_calf_left_joint: type revolute, parent autobed/quad_left_link, child autobed/calf_left_link, origin xyz=0.41218 0.11044 0 rpy=3.1416 8.5469E-14 -2.8798, axis 0 0 1, limit lower=-3. upper=3. effort=0 velocity=0
- added joint autobed/quad_calf_right_joint: type revolute, parent autobed/quad_right_link, child autobed/calf_right_link, origin xyz=0.41218 0.11044 0 rpy=3.1416 8.5225E-14 -2.8798, axis 0 0 1, limit lower=-3 upper=3 effort=0 velocity=0
- added joint autobed/tele_legs_joint: type prismatic, parent autobed/base_link, child autobed/bed_frame_link, origin xyz=-0.0400000000000005 0 0.320000000000001 rpy=0 0 0, axis 0 0 1, limit lower=-1 upper=1 effort=0 velocity=0
- added joint autobed/upper_mid_body_joint: type revolute, parent autobed/upper_body_link, child autobed/mid_body_link, origin xyz=0.35052 0 0 rpy=2.8327E-14 7.7949E-14 0.34907, axis 0 0 -1, limit lower=-2 upper=2 effort=0 velocity=0

File: hrl_base_selection/urdf/wheelchair_henry/robots/wheelchair_henry_head_position.URDF (robot description, URDF)
Before this commit: robot wheelchair_henry, 24 links, 23 joints
Links:
- removed link wheelchair/head_roty_link
- removed link wheelchair/head_rotz_link
- removed link wheelchair/neck_base_link
- removed link wheelchair/neck_tilt_link
- removed link wheelchair/neck_top_rotated_link
- removed link wheelchair/neck_twist_link
- added link wheelchair/neck_rotation; collision mesh filename=package://hrl_base_selection/urdf/wheelchair_henry/meshes/n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; visual mesh filename=package://hrl_base_selection/urdf/wheelchair_henry/meshes/n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
- link wheelchair/arm_left_link: geometry collision mesh filename=package://hrl_base_selection/urdf/wheelchair_henry/meshes/a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; visual mesh filename=package://hrl_base_selection/urdf/wheelchair_henry/meshes/a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
- link wheelchair/arm_right_link: geometry collision mesh filename=package://hrl_base_selection/urdf/wheelchair_henry/meshes/a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; visual mesh filename=package://hrl_base_selection/urdf/wheelchair_henry/meshes/a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
- link wheelchair/calf_left_link: geometry collision mesh filename=package://hrl_base_selection/urdf/wheelchair_henry/meshes/c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; visual mesh filename=package://hrl_base_selection/urdf/wheelchair_henry/meshes/c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
- link wheelchair/calf_right_link: geometry collision mesh filename=package://hrl_base_selection/urdf/wheelchair_henry/meshes/c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; visual mesh filename=package://hrl_base_selection/urdf/wheelchair_henry/meshes/c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
- link wheelchair/foot_left_link: geometry collision mesh filename=package://hrl_base_selection/urdf/wheelchair_henry/meshes/f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; visual mesh filename=package://hrl_base_selection/urdf/wheelchair_henry/meshes/f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
- link wheelchair/foot_right_link: geometry collision mesh filename=package://hrl_base_selection/urdf/wheelchair_henry/meshes/f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; visual mesh filename=package://hrl_base_selection/urdf/wheelchair_henry/meshes/f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
- link wheelchair/forearm_left_link: geometry collision mesh filename=package://hrl_base_selection/urdf/wheelchair_henry/meshes/f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; visual mesh filename=package://hrl_base_selection/urdf/wheelchair_henry/meshes/f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
- link wheelchair/forearm_right_link: geometry collision mesh filename=package://hrl_base_selection/urdf/wheelchair_henry/meshes/f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; visual mesh filename=package://hrl_base_selection/urdf/wheelchair_henry/meshes/f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
- link wheelchair/hand_left_link: geometry collision mesh filename=package://hrl_base_selection/urdf/wheelchair_henry/meshes/h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; visual mesh filename=package://hrl_base_selection/urdf/wheelchair_henry/meshes/h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
- link wheelchair/hand_right_link: geometry collision mesh filename=package://hrl_base_selection/urdf/wheelchair_henry/meshes/h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; visual mesh filename=package://hrl_base_selection/urdf/wheelchair_henry/meshes/h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
- link wheelchair/head_link: geometry collision mesh filename=package://hrl_base_selection/urdf/wheelchair_henry/meshes/h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; visual mesh filename=package://hrl_base_selection/urdf/wheelchair_henry/meshes/h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
- link wheelchair/lower_body_link: geometry collision mesh filename=package://hrl_base_selection/urdf/wheelchair_henry/meshes/l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; visual mesh filename=package://hrl_base_selection/urdf/wheelchair_henry/meshes/l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
- link wheelchair/mid_body_link: geometry collision mesh filename=package://hrl_base_selection/urdf/wheelchair_henry/meshes/m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; visual mesh filename=package://hrl_base_selection/urdf/wheelchair_henry/meshes/m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
- link wheelchair/neck_link: geometry collision mesh filename=package://hrl_base_selection/urdf/wheelchair_henry/meshes/n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; visual mesh filename=package://hrl_base_selection/urdf/wheelchair_henry/meshes/n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
- link wheelchair/quad_left_link: geometry collision mesh filename=package://hrl_base_selection/urdf/wheelchair_henry/meshes/q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; visual mesh filename=package://hrl_base_selection/urdf/wheelchair_henry/meshes/q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
- link wheelchair/quad_right_link: geometry collision mesh filename=package://hrl_base_selection/urdf/wheelchair_henry/meshes/q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; visual mesh filename=package://hrl_base_selection/urdf/wheelchair_henry/meshes/q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
- link wheelchair/upper_body_link: geometry collision mesh filename=package://hrl_base_selection/urdf/wheelchair_henry/meshes/u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; visual mesh filename=package://hrl_base_selection/urdf/wheelchair_henry/meshes/u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
Joints:
- removed joint wheelchair/neck_head_rotx_joint
- removed joint wheelchair/neck_head_roty_joint
- removed joint wheelchair/neck_head_rotz_joint
- removed joint wheelchair/neck_rotation_fixed_joint
- removed joint wheelchair/neck_tilt_joint
- removed joint wheelchair/neck_to_neck_top_joint
- removed joint wheelchair/neck_twist_joint
- removed joint wheelchair/origin_to_neck_base_joint
- added joint wheelchair/head_neck_joint1: type revolute, parent wheelchair/head_link, child wheelchair/neck_rotation, origin xyz=-0.0254 0 -0.08509 rpy=-1.5708 1.1345 -3.1416, axis 0 0 -1, limit lower=-2 upper=2 effort=0 velocity=0
- added joint wheelchair/head_neck_joint2: type revolute, parent wheelchair/neck_rotation, child wheelchair/neck_link, origin xyz=0 0 0 rpy=0 3.1554E-30 0, axis 0 0 1, limit lower=-2 upper=2 effort=0 velocity=0
- added joint wheelchair/origin_to_base_joint: type fixed, parent wheelchair/base_link, child wheelchair/head_link, origin xyz=0.452 0.0 1.35 rpy=0. 0.1 0., axis 0 0 0, limit lower=-2 upper=2 effort=0 velocity=0
- joint wheelchair/arm_forearm_left_joint: origin xyz=0.28174 -0.0106 -0.04953 rpy=0 0 0 -> xyz=0.28174 -0.0106 -0.04953 rpy=1.1849E-16 -8.3419E-14 -1.6268E-27
- joint wheelchair/arm_forearm_right_joint: origin xyz=0.28194 0 0.04953 rpy=0 0 0 -> xyz=0.28194 0 0.04953 rpy=2.6089E-19 -8.3342E-14 0.037607
- joint wheelchair/body_arm_left_joint: origin xyz=0.09652 0 -0.17526 rpy=0 0 0 -> xyz=0.09652 0 -0.17526 rpy=2.6872E-15 8.287E-14 0.033074
- joint wheelchair/body_arm_right_joint: origin xyz=0.09652 0 0.17526 rpy=0 0 0 -> xyz=0.09652 0 0.17526 rpy=-3.0757E-16 8.2843E-14 -0.0045332
- joint wheelchair/body_quad_left_joint: origin xyz=0.05207 0 -0.08636 rpy=0 0 -.25 -> xyz=0.05207 0 -0.08636 rpy=-3.1554E-30 -3.1554E-30 -2.7756E-17
- joint wheelchair/body_quad_right_joint: origin xyz=0.05207 0 0.08636 rpy=0 0 -.25 -> xyz=0.05207 0 0.08636 rpy=-3.1554E-30 -3.1554E-30 -2.7756E-17
- joint wheelchair/calf_foot_left_joint: origin xyz=-0.41279 -0.03188 0 rpy=0 0 0.09 -> xyz=-0.41279 -0.03188 0 rpy=2.4608E-16 9.411E-16 0.077076
- joint wheelchair/calf_foot_right_joint: origin xyz=-0.41279 -0.03188 0 rpy=0 0 0.09 -> xyz=-0.41279 -0.03188 0 rpy=3.3137E-27 3.7799E-26 0.077076
- joint wheelchair/forearm_hand_left_joint: origin xyz=0.25146 0 0 rpy=0 0 0 -> xyz=0.25146 0 0 rpy=1.3447E-16 8.3999E-14 1.6283E-27
- joint wheelchair/forearm_hand_right_joint: origin xyz=0.25146 0 0 rpy=0 0 0 -> xyz=0.25146 0 0 rpy=1.9364E-14 8.3335E-14 1.6151E-27
- joint wheelchair/mid_lower_body_joint: axis 0 0 1 -> 0 0 -1; origin xyz=0.15113 0 0 rpy=0 0 0 -> xyz=0.15113 0 0 rpy=-4.3091E-16 1.669E-15 -0.57779
- joint wheelchair/neck_body_joint: origin xyz=0.00 0 0 rpy=0 0 0 -> xyz=0.07239 0 0 rpy=-8.8242E-17 -8.2927E-14 0.66506; parent wheelchair/neck_base_link -> wheelchair/neck_link
- joint wheelchair/quad_calf_left_joint: origin xyz=0.41218 0.11044 0 rpy=3.14159 0 3.43 -> xyz=0.41218 0.11044 0 rpy=3.1416 8.5469E-14 -2.8798
- joint wheelchair/quad_calf_right_joint: origin xyz=0.41218 0.11044 0 rpy=3.14159 0 3.43 -> xyz=0.41218 0.11044 0 rpy=3.1416 8.5225E-14 -2.8798
- joint wheelchair/upper_mid_body_joint: axis 0 0 1 -> 0 0 -1; origin xyz=0.35052 0 0 rpy=0 0 0 -> xyz=0.35052 0 0 rpy=2.8327E-14 7.7949E-14 0.34907
