Commit message: fixed mannequin urdf for visualization during system use

File: hrl_base_selection/urdf/bed_and_environment_mannequin/robots/bed_and_environment_mannequin.urdf.xacro (robot description, xacro)
@@ -1,5 +1,5 @@
 <?xml version="1.0"?>
 <robot xmlns:xacro="http://www.ros.org/wiki/xacro" name="bed_and_environment_mannequin">
-<xacro:property name="body_len" value="1.9" />
+<xacro:property name="body_len" value="1.7" />
 <xacro:property name="comp_len" value="1.755" />
 <xacro:property name="torso_thickness" value="${body_len/comp_len*0.18}" />
@@ -332,5 +332,5 @@
     type="revolute">
     <origin
-      xyz="${rotated_torso+clavicle_len} ${0.15+0.21-0.04} 0"
+      xyz="${rotated_torso+clavicle_len} ${0.15+0.21-0.12} 0"
       rpy="0. 0. 0." />
     <!--<origin-->

Commit message: cleaning up some unneeded files

File: hrl_base_selection/urdf/bed_and_environment_mannequin/robots/bed_and_environment_mannequin.urdf.xacro (robot description, xacro)
@@ -12,6 +12,6 @@
 <xacro:property name="torso_len" value="${body_len/comp_len*0.460}" />
 <xacro:property name="leg_len" value="${body_len/comp_len*0.927}" />
-<xacro:property name="thigh_len" value="${body_len/comp_len*0.927}" />
-<xacro:property name="shank_len" value="${body_len/comp_len*0.927}" />
+<!--<xacro:property name="thigh_len" value="${body_len/comp_len*0.927}" />-->
+<!--<xacro:property name="shank_len" value="${body_len/comp_len*0.927}" />-->
 <xacro:property name="leg_len" value="${body_len/comp_len*0.927}" />
 <xacro:property name="upper_arm_len" value="${body_len/comp_len*0.279}" />
