Commit message: added STL files that were URDF dependencies

File: hrl_pose_estimation/urdf/bed_and_environment_henry_tray/robots/bed_and_environment_henry_tray.URDF (robot description, URDF)
Before this commit: robot bed_and_environment_henry_tray, 33 links, 32 joints
Links:
- link autobed/arm_left_link: geometry collision mesh filename=package://hrl_pose_estimation/urdf/bed_and_environment_henr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; visual mesh filename=package://hrl_pose_estimation/urdf/bed_and_environment_henr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
- link autobed/arm_right_link: geometry collision mesh filename=package://hrl_pose_estimation/urdf/bed_and_environment_henr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; visual mesh filename=package://hrl_pose_estimation/urdf/bed_and_environment_henr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
- link autobed/base_link: geometry collision mesh filename=package://hrl_pose_estimation/urdf/bed_and_environment_henr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; visual mesh filename=package://hrl_pose_estimation/urdf/bed_and_environment_henr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
- link autobed/bed_frame_link: geometry collision mesh filename=package://hrl_pose_estimation/urdf/bed_and_environment_henr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; visual mesh filename=package://hrl_pose_estimation/urdf/bed_and_environment_henr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
- link autobed/calf_left_link: geometry collision mesh filename=package://hrl_pose_estimation/urdf/bed_and_environment_henr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; visual mesh filename=package://hrl_pose_estimation/urdf/bed_and_environment_henr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
- link autobed/calf_right_link: geometry collision mesh filename=package://hrl_pose_estimation/urdf/bed_and_environment_henr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; visual mesh filename=package://hrl_pose_estimation/urdf/bed_and_environment_henr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
- link autobed/foot_left_link: geometry collision mesh filename=package://hrl_pose_estimation/urdf/bed_and_environment_henr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; visual mesh filename=package://hrl_pose_estimation/urdf/bed_and_environment_henr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
- link autobed/foot_right_link: geometry collision mesh filename=package://hrl_pose_estimation/urdf/bed_and_environment_henr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; visual mesh filename=package://hrl_pose_estimation/urdf/bed_and_environment_henr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
- link autobed/forearm_left_link: geometry collision mesh filename=package://hrl_pose_estimation/urdf/bed_and_environment_henr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; visual mesh filename=package://hrl_pose_estimation/urdf/bed_and_environment_henr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
- link autobed/forearm_right_link: geometry collision mesh filename=package://hrl_pose_estimation/urdf/bed_and_environment_henr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; visual mesh filename=package://hrl_pose_estimation/urdf/bed_and_environment_henr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
- link autobed/hand_left_link: geometry collision mesh filename=package://hrl_pose_estimation/urdf/bed_and_environment_henr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; visual mesh filename=package://hrl_pose_estimation/urdf/bed_and_environment_henr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
- link autobed/hand_right_link: geometry collision mesh filename=package://hrl_pose_estimation/urdf/bed_and_environment_henr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; visual mesh filename=package://hrl_pose_estimation/urdf/bed_and_environment_henr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
- link autobed/head_link: geometry collision mesh filename=package://hrl_pose_estimation/urdf/bed_and_environment_henr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; visual mesh filename=package://hrl_pose_estimation/urdf/bed_and_environment_henr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
- link autobed/head_rest_link: geometry collision mesh filename=package://hrl_pose_estimation/urdf/bed_and_environment_henr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; visual mesh filename=package://hrl_pose_estimation/urdf/bed_and_environment_henr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
- link autobed/leg_rest_lower: geometry collision mesh filename=package://hrl_pose_estimation/urdf/bed_and_environment_henr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; visual mesh filename=package://hrl_pose_estimation/urdf/bed_and_environment_henr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
- link autobed/leg_rest_upper: geometry collision mesh filename=package://hrl_pose_estimation/urdf/bed_and_environment_henr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; visual mesh filename=package://hrl_pose_estimation/urdf/bed_and_environment_henr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
- link autobed/lower_body_link: geometry collision mesh filename=package://hrl_pose_estimation/urdf/bed_and_environment_henr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; visual mesh filename=package://hrl_pose_estimation/urdf/bed_and_environment_henr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
- link autobed/mid_body_link: geometry collision mesh filename=package://hrl_pose_estimation/urdf/bed_and_environment_henr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; visual mesh filename=package://hrl_pose_estimation/urdf/bed_and_environment_henr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
- link autobed/neck_link: geometry collision mesh filename=package://hrl_pose_estimation/urdf/bed_and_environment_henr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; visual mesh filename=package://hrl_pose_estimation/urdf/bed_and_environment_henr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
- link autobed/quad_left_link: geometry collision mesh filename=package://hrl_pose_estimation/urdf/bed_and_environment_henr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; visual mesh filename=package://hrl_pose_estimation/urdf/bed_and_environment_henr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
- link autobed/quad_right_link: geometry collision mesh filename=package://hrl_pose_estimation/urdf/bed_and_environment_henr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; visual mesh filename=package://hrl_pose_estimation/urdf/bed_and_environment_henr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
- link autobed/upper_body_link: geometry collision mesh filename=package://hrl_pose_estimation/urdf/bed_and_environment_henr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; visual mesh filename=package://hrl_pose_estimation/urdf/bed_and_environment_henr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
- link autobed/wall_link: geometry collision mesh filename=package://hrl_pose_estimation/urdf/bed_and_environment_henr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; visual mesh filename=package://hrl_pose_estimation/urdf/bed_and_environment_henr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
