Commit message: saving chnages to urdf from things at henrys house

File: hrl_base_selection/urdf/bed_and_environment_cali_henry_tray/robots/bed_and_environment_cali_1_9m_tray.URDF (robot description, URDF)
Before this commit: robot bed_and_environment_cali_parameterized_tray, 43 links, 42 joints
Joints:
- joint autobed/head_rest_hinge: origin xyz=0.835 0 0.21 rpy=1.5708 0 -3.1416 -> xyz=0.835 0 0.04 rpy=1.5708 0 -3.1416
- joint autobed/headrest_bed_to_worldframe_joint: origin xyz=0.41 0.15 0 rpy=0. 0. 0. -> xyz=0.41 0.32 0 rpy=0. 0. 0.

File: hrl_base_selection/urdf/bed_and_environment_cali_henry_tray/robots/bed_and_environment_cali_1_9m_tray_openrave.URDF (robot description, URDF)
Before this commit: robot bed_and_environment_cali_parameterized_tray, 43 links, 42 joints
Joints:
- joint autobed/head_rest_hinge: origin xyz=0.835 0 0.21 rpy=1.5708 0 -3.1416 -> xyz=0.835 0 0.04 rpy=1.5708 0 -3.1416
- joint autobed/headrest_bed_to_worldframe_joint: origin xyz=0.41 0.15 0 rpy=0. 0. 0. -> xyz=0.41 0.32 0 rpy=0. 0. 0.

File: hrl_base_selection/urdf/bed_and_environment_cali_henry_tray/robots/bed_and_environment_cali_parameterized_tray.URDF (robot description, URDF)
Before this commit: robot bed_and_environment_cali_parameterized_tray, 43 links, 42 joints
Joints:
- joint autobed/head_rest_hinge: origin xyz=0.835 0 0.21 rpy=1.5708 0 -3.1416 -> xyz=0.835 0 0.04 rpy=1.5708 0 -3.1416
- joint autobed/headrest_bed_to_worldframe_joint: origin xyz=0.41 0.15 0 rpy=0. 0. 0. -> xyz=0.41 0.32 0 rpy=0. 0. 0.

File: hrl_base_selection/urdf/bed_and_environment_cali_henry_tray/robots/bed_and_environment_cali_parameterized_tray_openrave.URDF (robot description, URDF)
Before this commit: robot bed_and_environment_cali_parameterized_tray, 43 links, 42 joints
Joints:
- joint autobed/head_rest_hinge: origin xyz=0.835 0 0.21 rpy=1.5708 0 -3.1416 -> xyz=0.835 0 0.04 rpy=1.5708 0 -3.1416
- joint autobed/headrest_bed_to_worldframe_joint: origin xyz=0.41 0.15 0 rpy=0. 0. 0. -> xyz=0.41 0.32 0 rpy=0. 0. 0.
