Commit message: changes to include and exclude bed movement and head movement for toc and baseline methods. also expanded model via scaling and via adjusting meshes. also now for single configuration will try initializing on each side of the bed. this makes comparisons more fair.

File: hrl_base_selection/urdf/autobed_simulation/robots/autobed_simulation_expanded.URDF (robot description, URDF)
Before this commit: robot autobed_simulation_expanded, 33 links, 32 joints
Links:
- link autobed/arm_left_link: geometry collision mesh filename=package://hrl_base_selection/urdf/autobed_simulation/meshes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 scale=1.0 1.3 1.3; visual mesh filename=package://hrl_base_selection/urdf/autobed_simulation/meshes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 scale=1.0 1.3 1.3
- link autobed/arm_right_link: geometry collision mesh filename=package://hrl_base_selection/urdf/autobed_simulation/meshes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 scale=1.0 1.3 1.3; visual mesh filename=package://hrl_base_selection/urdf/autobed_simulation/meshes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 scale=1.0 1.3 1.3
- link autobed/calf_left_link: geometry collision mesh filename=package://hrl_base_selection/urdf/autobed_simulation/meshes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 scale=1.0 1.3 1.3; visual mesh filename=package://hrl_base_selection/urdf/autobed_simulation/meshes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 scale=1.0 1.3 1.3
- link autobed/calf_right_link: geometry collision mesh filename=package://hrl_base_selection/urdf/autobed_simulation/meshes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 scale=1.0 1.3 1.3; visual mesh filename=package://hrl_base_selection/urdf/autobed_simulation/meshes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 scale=1.0 1.3 1.3
- link autobed/foot_left_link: geometry collision mesh filename=package://hrl_base_selection/urdf/autobed_simulation/meshes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 scale=1.5 1.2 1.5; visual mesh filename=package://hrl_base_selection/urdf/autobed_simulation/meshes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 scale=1.5 1.2 1.5
- link autobed/foot_right_link: geometry collision mesh filename=package://hrl_base_selection/urdf/autobed_simulation/meshes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 scale=1.5 1.2 1.5; visual mesh filename=package://hrl_base_selection/urdf/autobed_simulation/meshes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 scale=1.5 1.2 1.5
- link autobed/forearm_left_link: geometry collision mesh filename=package://hrl_base_selection/urdf/autobed_simulation/meshes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 scale=1.0 1.3 1.3; visual mesh filename=package://hrl_base_selection/urdf/autobed_simulation/meshes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 scale=1.0 1.3 1.3
- link autobed/forearm_right_link: geometry collision mesh filename=package://hrl_base_selection/urdf/autobed_simulation/meshes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 scale=1.0 1.3 1.3; visual mesh filename=package://hrl_base_selection/urdf/autobed_simulation/meshes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 scale=1.0 1.3 1.3
- link autobed/hand_left_link: geometry collision mesh filename=package://hrl_base_selection/urdf/autobed_simulation/meshes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 scale=1.0 1.3 1.3; visual mesh filename=package://hrl_base_selection/urdf/autobed_simulation/meshes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 scale=1.0 1.3 1.3
- link autobed/hand_right_link: geometry collision mesh filename=package://hrl_base_selection/urdf/autobed_simulation/meshes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 scale=1.0 1.3 1.3; visual mesh filename=package://hrl_base_selection/urdf/autobed_simulation/meshes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 scale=1.0 1.3 1.3
- link autobed/head_link: geometry collision mesh filename=package://hrl_base_selection/urdf/autobed_simulation/meshes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 scale=1.1 1.1 1.1; visual mesh filename=package://hrl_base_selection/urdf/autobed_simulation/meshes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 scale=1.1 1.1 1.1
- link autobed/head_rest_link: geometry collision mesh filename=package://hrl_base_selection/urdf/autobed_simulation/meshes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 scale=1.0 1.3 1.3; visual mesh filename=package://hrl_base_selection/urdf/autobed_simulation/meshes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
- link autobed/lower_body_link: geometry collision mesh filename=package://hrl_base_selection/urdf/autobed_simulation/meshes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 scale=1.0 1.3 1.3; visual mesh filename=package://hrl_base_selection/urdf/autobed_simulation/meshes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 scale=1.0 1.3 1.3
- link autobed/mid_body_link: geometry collision mesh filename=package://hrl_base_selection/urdf/autobed_simulation/meshes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 scale=1.0 1.3 1.3; visual mesh filename=package://hrl_base_selection/urdf/autobed_simulation/meshes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 scale=1.0 1.3 1.3
- link autobed/neck_link: geometry collision mesh filename=package://hrl_base_selection/urdf/autobed_simulation/meshes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 scale=1.0 1.3 1.3; visual mesh filename=package://hrl_base_selection/urdf/autobed_simulation/meshes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 scale=1.0 1.3 1.3
- link autobed/quad_left_link: geometry collision mesh filename=package://hrl_base_selection/urdf/autobed_simulation/meshes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 scale=1.0 1.3 1.3; visual mesh filename=package://hrl_base_selection/urdf/autobed_simulation/meshes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 scale=1.0 1.3 1.3
- link autobed/quad_right_link: geometry collision mesh filename=package://hrl_base_selection/urdf/autobed_simulation/meshes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 scale=1.0 1.3 1.3; visual mesh filename=package://hrl_base_selection/urdf/autobed_simulation/meshes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 scale=1.0 1.3 1.3
- link autobed/upper_body_link: geometry collision mesh filename=package://hrl_base_selection/urdf/autobed_simulation/meshes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 scale=1.0 1.3 1.3; visual mesh filename=package://hrl_base_selection/urdf/autobed_simulation/meshes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 scale=1.0 1.3 1.3
Joints:
- joint autobed/origin_wall_joint: axis 0 0 0 -> 0.984220866265583 0.172903665695305 0.0375979892620764; limit (none) -> lower=-3 upper=3 effort=0 velocity=0; type fixed -> prismatic

File: hrl_base_selection/urdf/autobed_simulation/robots/autobed_simulation_normal.URDF (robot description, URDF)
Before this commit: robot autobed_simulation_normal, 33 links, 32 joints
Joints:
- joint autobed/origin_wall_joint: axis 0 0 0 -> 0.984220866265583 0.172903665695305 0.0375979892620764; limit (none) -> lower=-3 upper=3 effort=0 velocity=0; type fixed -> prismatic

File: hrl_base_selection/urdf/wheelchair_simulation/robots/wheelchair_simulation_expanded.URDF (robot description, URDF)
Before this commit: robot wheelchair_simulation_expanded, 27 links, 26 joints
Links:
- link wheelchair/arm_left_link: geometry collision mesh filename=package://hrl_base_selection/urdf/wheelchair_simulation/mes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 scale=1.0 1.3 1.3; visual mesh filename=package://hrl_base_selection/urdf/wheelchair_simulation/mes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 scale=1.0 1.3 1.3
- link wheelchair/arm_right_link: geometry collision mesh filename=package://hrl_base_selection/urdf/wheelchair_simulation/mes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 scale=1.0 1.3 1.3; visual mesh filename=package://hrl_base_selection/urdf/wheelchair_simulation/mes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 scale=1.0 1.3 1.3
- link wheelchair/calf_left_link: geometry collision mesh filename=package://hrl_base_selection/urdf/wheelchair_simulation/mes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 scale=1.0 1.3 1.3; visual mesh filename=package://hrl_base_selection/urdf/wheelchair_simulation/mes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 scale=1.0 1.3 1.3
- link wheelchair/calf_right_link: geometry collision mesh filename=package://hrl_base_selection/urdf/wheelchair_simulation/mes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 scale=1.0 1.3 1.3; visual mesh filename=package://hrl_base_selection/urdf/wheelchair_simulation/mes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 scale=1.0 1.3 1.3
- link wheelchair/foot_left_link: geometry collision mesh filename=package://hrl_base_selection/urdf/wheelchair_simulation/mes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 scale=1.5 1.2 1.5; visual mesh filename=package://hrl_base_selection/urdf/wheelchair_simulation/mes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 scale=1.5 1.2 1.5
- link wheelchair/foot_right_link: geometry collision mesh filename=package://hrl_base_selection/urdf/wheelchair_simulation/mes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 scale=1.5 1.2 1.5; visual mesh filename=package://hrl_base_selection/urdf/wheelchair_simulation/mes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 scale=1.5 1.2 1.5
- link wheelchair/forearm_left_link: geometry collision mesh filename=package://hrl_base_selection/urdf/wheelchair_simulation/mes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 scale=1.0 1.3 1.3; visual mesh filename=package://hrl_base_selection/urdf/wheelchair_simulation/mes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 scale=1.0 1.3 1.3
- link wheelchair/forearm_right_link: geometry collision mesh filename=package://hrl_base_selection/urdf/wheelchair_simulation/mes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 scale=1.0 1.3 1.3; visual mesh filename=package://hrl_base_selection/urdf/wheelchair_simulation/mes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 scale=1.0 1.3 1.3
- link wheelchair/hand_left_link: geometry collision mesh filename=package://hrl_base_selection/urdf/wheelchair_simulation/mes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 scale=1.0 1.3 1.3; visual mesh filename=package://hrl_base_selection/urdf/wheelchair_simulation/mes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 scale=1.0 1.3 1.3
- link wheelchair/hand_right_link: geometry collision mesh filename=package://hrl_base_selection/urdf/wheelchair_simulation/mes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 scale=1.0 1.3 1.3; visual mesh filename=package://hrl_base_selection/urdf/wheelchair_simulation/mes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 scale=1.0 1.3 1.3
- link wheelchair/head_link: geometry collision mesh filename=package://hrl_base_selection/urdf/wheelchair_simulation/mes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 scale=1.1 1.1 1.1; visual mesh filename=package://hrl_base_selection/urdf/wheelchair_simulation/mes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 scale=1.1 1.1 1.1
- link wheelchair/lower_body_link: geometry collision mesh filename=package://hrl_base_selection/urdf/wheelchair_simulation/mes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 scale=1.0 1.3 1.3; visual mesh filename=package://hrl_base_selection/urdf/wheelchair_simulation/mes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 scale=1.0 1.3 1.3
- link wheelchair/mid_body_link: geometry collision mesh filename=package://hrl_base_selection/urdf/wheelchair_simulation/mes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 scale=1.0 1.3 1.3; visual mesh filename=package://hrl_base_selection/urdf/wheelchair_simulation/mes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 scale=1.0 1.3 1.3
- link wheelchair/neck_link: geometry collision mesh filename=package://hrl_base_selection/urdf/wheelchair_simulation/mes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 scale=1.0 1.3 1.3; visual mesh filename=package://hrl_base_selection/urdf/wheelchair_simulation/mes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 scale=1.0 1.3 1.3
- link wheelchair/quad_left_link: geometry collision mesh filename=package://hrl_base_selection/urdf/wheelchair_simulation/mes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 scale=1.0 1.3 1.3; visual mesh filename=package://hrl_base_selection/urdf/wheelchair_simulation/mes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 scale=1.0 1.3 1.3
- link wheelchair/quad_right_link: geometry collision mesh filename=package://hrl_base_selection/urdf/wheelchair_simulation/mes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 scale=1.0 1.3 1.3; visual mesh filename=package://hrl_base_selection/urdf/wheelchair_simulation/mes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 scale=1.0 1.3 1.3
- link wheelchair/upper_body_link: geometry collision mesh filename=package://hrl_base_selection/urdf/wheelchair_simulation/mes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 scale=1.0 1.3 1.3; visual mesh filename=package://hrl_base_selection/urdf/wheelchair_simulation/mes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 scale=1.0 1.3 1.3

Commit message: made head normal size

File: hrl_base_selection/urdf/autobed_simulation/robots/autobed_simulation_expanded.URDF (robot description, URDF)
Before this commit: robot autobed_simulation_expanded, 33 links, 32 joints
Links:
- link autobed/head_link: geometry collision mesh filename=package://hrl_base_selection/urdf/autobed_simulation/meshes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 scale=1.0 1.0 1.0; visual mesh filename=package://hrl_base_selection/urdf/autobed_simulation/meshes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 scale=1.0 1.0 1.0

File: hrl_base_selection/urdf/wheelchair_simulation/robots/wheelchair_simulation_expanded.URDF (robot description, URDF)
Before this commit: robot wheelchair_simulation_expanded, 27 links, 26 joints
Links:
- link wheelchair/head_link: geometry collision mesh filename=package://hrl_base_selection/urdf/wheelchair_simulation/mes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 scale=1. 1. 1.; visual mesh filename=package://hrl_base_selection/urdf/wheelchair_simulation/mes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 scale=1. 1. 1.
