Commit message: commiting so i can switch branches

File: hrl_base_selection/models/gown_box_only.urdf (robot description, URDF)
Before this commit: robot gown_box, 1 links, 0 joints
Links:
- link gown: geometry collision box size=0.04 0.12 0.25; visual box size=0.04 0.12 0.25

Commit message: added wheelchair

File: hrl_base_selection/models/gown_box_only.urdf (robot description, URDF)
Before this commit: robot gown_box, 1 links, 0 joints
Links:
- link gown: geometry collision box size=0.08 0.12 0.3; visual box size=0.08 0.12 0.3
