Commit message: [ari_dart_devel] Committing all things so it can be released.

File: hrl_base_selection/urdf/bed_and_body_v3_real_expanded/robots/bed_and_body_v3_with_wall.URDF (robot description, URDF)
Before this commit: robot bed_and_body_v3, 26 links, 25 joints
Links:
- link arm_left_link: geometry collision mesh filename=package://hrl_base_selection/urdf/bed_and_body_v3_real_expa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; visual mesh filename=package://hrl_base_selection/urdf/bed_and_body_v3_real_expa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
- link arm_right_link: geometry collision mesh filename=package://hrl_base_selection/urdf/bed_and_body_v3_real_expa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; visual mesh filename=package://hrl_base_selection/urdf/bed_and_body_v3_real_expa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
- link base_link: geometry collision mesh filename=package://hrl_base_selection/urdf/bed_and_body_v3_real_expa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; visual mesh filename=package://hrl_base_selection/urdf/bed_and_body_v3_real_expa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
- link bed_frame_link: geometry collision mesh filename=package://hrl_base_selection/urdf/bed_and_body_v3_real_expa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; visual mesh filename=package://hrl_base_selection/urdf/bed_and_body_v3_real_expa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
- link calf_left_link: geometry collision mesh filename=package://hrl_base_selection/urdf/bed_and_body_v3_real_expa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; visual mesh filename=package://hrl_base_selection/urdf/bed_and_body_v3_real_expa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
- link calf_right_link: geometry collision mesh filename=package://hrl_base_selection/urdf/bed_and_body_v3_real_expa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; visual mesh filename=package://hrl_base_selection/urdf/bed_and_body_v3_real_expa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
- link foot_left_link: geometry collision mesh filename=package://hrl_base_selection/urdf/bed_and_body_v3_real_expa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; visual mesh filename=package://hrl_base_selection/urdf/bed_and_body_v3_real_expa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
- link foot_right_link: geometry collision mesh filename=package://hrl_base_selection/urdf/bed_and_body_v3_real_expa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; visual mesh filename=package://hrl_base_selection/urdf/bed_and_body_v3_real_expa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
- link forearm_left_link: geometry collision mesh filename=package://hrl_base_selection/urdf/bed_and_body_v3_real_expa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; visual mesh filename=package://hrl_base_selection/urdf/bed_and_body_v3_real_expa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
- link forearm_right_link: geometry collision mesh filename=package://hrl_base_selection/urdf/bed_and_body_v3_real_expa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; visual mesh filename=package://hrl_base_selection/urdf/bed_and_body_v3_real_expa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
- link hand_left_link: geometry collision mesh filename=package://hrl_base_selection/urdf/bed_and_body_v3_real_expa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; visual mesh filename=package://hrl_base_selection/urdf/bed_and_body_v3_real_expa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
- link hand_right_link: geometry collision mesh filename=package://hrl_base_selection/urdf/bed_and_body_v3_real_expa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; visual mesh filename=package://hrl_base_selection/urdf/bed_and_body_v3_real_expa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
- link head_link: geometry collision mesh filename=package://hrl_base_selection/urdf/bed_and_body_v3_real_expa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; visual mesh filename=package://hrl_base_selection/urdf/bed_and_body_v3_real_expa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
- link head_rest_link: geometry collision mesh filename=package://hrl_base_selection/urdf/bed_and_body_v3_real_expa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; visual mesh filename=package://hrl_base_selection/urdf/bed_and_body_v3_real_expa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
- link leg_rest_lower_link: geometry collision mesh filename=package://hrl_base_selection/urdf/bed_and_body_v3_real_expa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; visual mesh filename=package://hrl_base_selection/urdf/bed_and_body_v3_real_expa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
- link leg_rest_upper_link: geometry collision mesh filename=package://hrl_base_selection/urdf/bed_and_body_v3_real_expa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; visual mesh filename=package://hrl_base_selection/urdf/bed_and_body_v3_real_expa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
- link lower_body_link: geometry collision mesh filename=package://hrl_base_selection/urdf/bed_and_body_v3_real_expa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; visual mesh filename=package://hrl_base_selection/urdf/bed_and_body_v3_real_expa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
- link mid_body_link: geometry collision mesh filename=package://hrl_base_selection/urdf/bed_and_body_v3_real_expa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; visual mesh filename=package://hrl_base_selection/urdf/bed_and_body_v3_real_expa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
- link neck_link: geometry collision mesh filename=package://hrl_base_selection/urdf/bed_and_body_v3_real_expa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; visual mesh filename=package://hrl_base_selection/urdf/bed_and_body_v3_real_expa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
- link neck_rotation: geometry collision mesh filename=package://hrl_base_selection/urdf/bed_and_body_v3_real_expa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; visual mesh filename=package://hrl_base_selection/urdf/bed_and_body_v3_real_expa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
- link quad_left_link: geometry collision mesh filename=package://hrl_base_selection/urdf/bed_and_body_v3_real_expa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; visual mesh filename=package://hrl_base_selection/urdf/bed_and_body_v3_real_expa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
- link quad_right_link: geometry collision mesh filename=package://hrl_base_selection/urdf/bed_and_body_v3_real_expa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; visual mesh filename=package://hrl_base_selection/urdf/bed_and_body_v3_real_expa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
- link upper_body_link: geometry collision mesh filename=package://hrl_base_selection/urdf/bed_and_body_v3_real_expa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; visual mesh filename=package://hrl_base_selection/urdf/bed_and_body_v3_real_expa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
- link wall_link: geometry collision mesh filename=package://hrl_base_selection/urdf/bed_and_body_v3_real_expa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; visual mesh filename=package://hrl_base_selection/urdf/bed_and_body_v3_real_expa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

File: hrl_base_selection/urdf/wheelchair_and_body_assembly/robots/wheelchair_and_body_assembly.URDF (robot description, URDF)
Before this commit: robot wheelchair_and_body_assembly, 5 links, 4 joints
Links:
- removed link base_link
- removed link body_th_move_link
- removed link body_x_move_link
- removed link body_y_move_link
- removed link head_center
- added link wheelchair/base_link, mass 63.649; collision mesh filename=package://hrl_base_selection/urdf/wheelchair_and_body_assem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; visual mesh filename=package://hrl_base_selection/urdf/wheelchair_and_body_assem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
- added link wheelchair/body_th_move_link, mass 55.001
- added link wheelchair/body_x_move_link, mass 55.0007697502791
- added link wheelchair/body_y_move_link, mass 55.001; collision meshZZZZZZZZZ filename=package://hrl_base_selection/urdf/wheelchair_and_body_assem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; visual mesh filename=package://hrl_base_selection/urdf/wheelchair_and_body_assem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
- added link wheelchair/head_center, mass 3.93285195403502; collision mesh filename=package://hrl_base_selection/urdf/wheelchair_and_body_assem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; visual mesh filename=package://hrl_base_selection/urdf/wheelchair_and_body_assem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
Joints:
- removed joint head_neck_joint
- removed joint wheelchair_body_rotation_joint
- removed joint wheelchair_body_x_joint
- removed joint wheelchair_body_y_joint
- added joint wheelchair/head_neck_joint: type revolute, parent body_y_move_link, child head_center, origin xyz=0.048166 0 0.76169 rpy=0 0 0, axis 0 -1 0, limit lower=-2 upper=2 effort=0 velocity=0
- added joint wheelchair/wheelchair_body_rotation_joint: type revolute, parent base_link, child body_th_move_link, origin xyz=0.40278 0 0.47 rpy=0 0 0, axis 0 0 -1, limit lower=-1 upper=1 effort=0 velocity=0
- added joint wheelchair/wheelchair_body_x_joint: type prismatic, parent body_th_move_link, child body_x_move_link, origin xyz=0 0 0 rpy=0 0 0, axis -1 0 0, limit lower=-1 upper=1 effort=0 velocity=0
- added joint wheelchair/wheelchair_body_y_joint: type prismatic, parent body_x_move_link, child body_y_move_link, origin xyz=0 0 0 rpy=0 0 0, axis 0 -1 0, limit lower=-1 upper=1 effort=0 velocity=0

File: hrl_base_selection/urdf/wheelchair_henry/robots/wheelchair_henry.URDF (robot description, URDF)
Before this commit: robot wheelchair_henry, 24 links, 23 joints
Links:
- added link wheelchair/body_theta_move_link
- added link wheelchair/body_x_move_link
- added link wheelchair/body_y_move_link
Joints:
- added joint wheelchair/body_theta_move_joint: type revolute, parent wheelchair/body_y_move_link, child wheelchair/body_theta_move_link, origin xyz=0.0 0.0 0.0 rpy=0 0 0, axis 0 0 1, limit lower=-3 upper=3 effort=0 velocity=0
- added joint wheelchair/body_x_move_joint: type prismatic, parent wheelchair/base_link, child wheelchair/body_x_move_link, origin xyz=0.332 0 1.25 rpy=0 0 0, axis 1 0 0, limit lower=-1 upper=1 effort=0 velocity=0
- added joint wheelchair/body_y_move_joint: type prismatic, parent wheelchair/body_x_move_link, child wheelchair/body_y_move_link, origin xyz=0.0 0.0 0.0 rpy=0 0 0, axis 0 1 0, limit lower=-1 upper=1 effort=0 velocity=0
- joint wheelchair/origin_to_neck_base_joint: origin xyz=0.332 0 1.25 rpy=1.570795 1.570795 0 -> xyz=0.0 0.0 0.0 rpy=1.570795 1.570795 0; parent wheelchair/base_link -> wheelchair/body_theta_move_link
